File: MotorController.sch (KiCad schematic (older format))
At the start: 36 parts, among them J1 Conn_01x03_Male, J2 Conn_01x05_Female, J3 Conn_01x03_Male, J4 Conn_01x03_Female, U10 FDD3672, U11 FDD3672, U12 FDD3672, U13 FDD3672, U3 FDD3672, U4 FDD3672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

Commit message: Syncing for travel
Parts:
- removed J3: Conn_01x03_Male, Connector_Molex:Molex_KK-254_AE-6410-03A_1x03_P2.54mm_Vertical, symbol Connector:Conn_01x03_Male
- added C? (x3): 0.1uF, symbol Device:C_Small
- added J? (x2): Conn_01x02_Male, symbol Connector:Conn_01x02_Male
- added R?: NP, symbol Device:R_Small_US
- added U?: ATtiny814-SS, Package_SO:SOIC-14_3.9x8.7mm_P1.27mm, symbol MCU_Microchip_ATtiny:ATtiny814-SS
- added U?: MCP2515-xSO, Package_SO:SOIC-18W_7.5x11.6mm_P1.27mm, symbol Interface_CAN_LIN:MCP2515-xSO
- added U?: TJA1051T-E, Package_SO:SOIC-8_3.9x4.9mm_P1.27mm, symbol Interface_CAN_LIN:TJA1051T-E
- U10, U11, U12, U13, U3, U4: symbol Mosfet:FDD3672 -> MotorController-rescue:FDD3672-Mosfet
- U7: symbol A4915:A4915MLPTR-T -> MotorController-rescue:A4915MLPTR-T-A4915
Connections:
- net GND: now also D1.1 (K)
- net VCC: now also R13.1; no longer D1.2 (A)
- net GLA: now reaches R9.1, U7.10 (GLA)
- net GHA: now reaches R11.1, U7.11 (GHA)
- net GLC: now reaches R10.1, U7.2 (GLC)
- net at R13.2, U7.22 (Fault): now also D1.2 (A)
- net ENABLE: now reaches U7.23 (Enable)
- net DIR: now reaches U7.24 (DIR)
- net BREAKn: now reaches U7.25 (BRAKEn)
- net HALL_A: now reaches J2.4 (Pin_4), U7.26 (HA)
- net HALL_B: now reaches J2.3 (Pin_3), U7.27 (HB)
- net HALL_C: now reaches J2.2 (Pin_2), U7.28 (HC)
- net GHC: now reaches R12.1, U7.3 (GHC)
- net GLB: now reaches R3.1, U7.6 (GLB)
- net GHB: now reaches R4.1, U7.7 (GHB)
- new net: U?.1 (TXCAN), U?.4 (RXD)
- new net: U?.1 (TXD), U?.2 (RXCAN)
- new net CAN_H: J?.2 (Pin_2), J?.2 (Pin_2), R?.1, U?.7 (CANH)
- new net CAN_L: J?.1 (Pin_1), J?.1 (Pin_1), R?.2, U?.6 (CANL)
- new net SPI_MISO: U?.12 (PA2), U?.15 (SO)
- new net SPI_MOSI: U?.11 (PA1), U?.14 (SI)
- new net SPI_SCK: U?.13 (PA3), U?.13 (SCK)
Other:
- note added: "CAN Communications"
- note added: "Hall effect sensor feedback"
- note added: "Motor Driver Controller"
- note added: "Motor Driver Half Bridges"
- note added: "Populate with 120 Ohm to terminate\nCAN bus at motor controller"
- note added: "TODO resistor too small?"
- moved on the sheet: C1, C2, C3, C4, C5, C6, C7, C8, C9, D1, D2, J1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

Commit message: I'm too tired to write a good message
Connections:
- net GND: now also C?.2, C?.2, C?.2, U?.14 (GND), U?.2 (GND), U?.9 (VSS)
- net VCC: now also C?.1, C?.1, C?.1, U?.1 (VCC), U?.18 (VDD), U?.3 (VCC)
- net CAN_SILENT: now reaches U?.5 (EN)
- net CAN_EN: now reaches U?.8 (S)
Other:
- moved on the sheet: C?, R?
Changed lines of the file:
@@
 Connection ~ 3900 5500
-$Comp
-L Interface_CAN_LIN:MCP2515-xSO U?
-U 1 1 5F40DB1B
-P 9200 2100
-F 0 "U?" H 9200 3081 50  0000 C CNN
-F 1 "MCP2515-xSO" H 9200 2990 50  0000 C CNN
-F 2 "Package_SO:SOIC-18W_7.5x11.6mm_P1.27mm" H 9200 1200 50  0001 C CIN
-F 3 "http://ww1.microchip.com/downloads/en/DeviceDoc/21801e.pdf" H 9300 1300 50  0001 C CNN
-	1    9200 2100
-	1    0    0    -1
-$EndComp
 $Comp
 L Interface_CAN_LIN:TJA1051T-E U?
 U 1 1 5F412D3F
 P 11300 1700
-F 0 "U?" H 11300 2281 50  0000 C CNN
-F 1 "TJA1051T-E" H 11300 2190 50  0000 C CNN
+F 0 "U?" H 10950 2050 50  0000 C CNN
+F 1 "TJA1051T-E" H 11600 2050 50  0000 C CNN
 F 2 "Package_SO:SOIC-8_3.9x4.9mm_P1.27mm" H 11300 1200 50  0001 C CIN
 F 3 "http://www.nxp.com/documents/data_sheet/TJA1051.pdf" H 11300 1700 50  0001 C CNN
@@
 Wire Wire Line
 	9800 1500 10800 1500
-Wire Wire Line
-	9800 1600 10800 1600
 $Comp
 L Connector:Conn_01x02_Male J?
@@
 L Device:R_Small_US R?
 U 1 1 5F03DAFA
-P 12250 2550
-F 0 "R?" H 12318 2596 50  0000 L CNN
-F 1 "NP" H 12318 2505 50  0000 L CNN
-F 2 "" H 12250 2550 50  0001 C CNN
-F 3 "~" H 12250 2550 50  0001 C CNN
-	1    12250 2550
-	1    0    0    -1
-$EndComp
-Wire Wire Line
-	12250 2450 12250 2350
-Wire Wire Line
-	12250 2350 12550 2350
-Wire Wire Line
-	12250 2650 12250 2800
-Text Label 12550 2350 2    50   ~ 0
+P 12900 2500
+F 0 "R?" H 12968 2546 50  0000 L CNN
+F 1 "NP" H 12968 2455 50  0000 L CNN
+F 2 "" H 12900 2500 50  0001 C CNN
+F 3 "~" H 12900 2500 50  0001 C CNN
+	1    12900 2500
+	1    0    0    -1
+$EndComp
+Wire Wire Line
+	12900 2400 12900 2300
+Wire Wire Line
+	12900 2300 13200 2300
+Wire Wire Line
+	12900 2600 12900 2750
+Text Label 13200 2300 2    50   ~ 0
 CAN_H
 Wire Wire Line
-	12250 2800 12550 2800
-Text Label 12550 2800 2    50   ~ 0
+	12900 2750 13200 2750
+Text Label 13200 2750 2    50   ~ 0
 CAN_L
-Text Notes 12600 2600 0    50   ~ 0
+Text Notes 13250 2550 0    50   ~ 0
 Populate with 120 Ohm to terminate\nCAN bus at motor controller
 $Comp
@@
 U 1 1 5F0D24D7
 P 10400 5150
-F 0 "U?" H 10400 6031 50  0000 C CNN
-F 1 "ATtiny814-SS" H 10400 5940 50  0000 C CNN
+F 0 "U?" H 10650 5800 50  0000 C CNN
+F 1 "ATtiny814-SS" H 10050 5800 50  0000 C CNN
 F 2 "Package_SO:SOIC-14_3.9x8.7mm_P1.27mm" H 10400 5150 50  0001 C CIN
 F 3 "http://ww1.microchip.com/downloads/en/DeviceDoc/40001912A.pdf" H 10400 5150 50  0001 C CNN
 	1    10400 5150
-	1    0    0    -1
-$EndComp
-$Comp
-L Device:C_Small C?
-U 1 1 5F0DAE10
-P 11400 4000
-F 0 "C?" H 11492 4046 50  0000 L CNN
-F 1 "0.1uF" H 11492 3955 50  0000 L CNN
-F 2 "" H 11400 4000 50  0001 C CNN
-F 3 "~" H 11400 4000 50  0001 C CNN
-	1    11400 4000
 	1    0    0    -1
 $EndComp
@@
 L Device:C_Small C?
 U 1 1 5F1B7761
-P 9900 1150
-F 0 "C?" H 9992 1196 50  0000 L CNN
-F 1 "0.1uF" H 9992 1105 50  0000 L CNN
-F 2 "" H 9900 1150 50  0001 C CNN
-F 3 "~" H 9900 1150 50  0001 C CNN
-	1    9900 1150
+P 8450 3300
+F 0 "C?" H 8542 3346 50  0000 L CNN
+F 1 "0.1uF" H 8542 3255 50  0000 L CNN
+F 2 "" H 8450 3300 50  0001 C CNN
+F 3 "~" H 8450 3300 50  0001 C CNN
+	1    8450 3300
 	1    0    0    -1
 $EndComp
@@
 L Device:C_Small C?
 U 1 1 5F1BFD1D
-P 11900 1100
-F 0 "C?" H 11992 1146 50  0000 L CNN
-F 1 "0.1uF" H 11992 1055 50  0000 L CNN
-F 2 "" H 11900 1100 50  0001 C CNN
-F 3 "~" H 11900 1100 50  0001 C CNN
-	1    11900 1100
+P 10750 2500
+F 0 "C?" H 10842 2546 50  0000 L CNN
+F 1 "0.1uF" H 10842 2455 50  0000 L CNN
+F 2 "" H 10750 2500 50  0001 C CNN
+F 3 "~" H 10750 2500 50  0001 C CNN
+	1    10750 2500
 	1    0    0    -1
 $EndComp
@@
 Wire Wire Line
 	6550 6400 6550 6300
+Wire Wire Line
+	10800 1800 10350 1800
+Wire Wire Line
+	10350 1900 10800 1900
+Text Label 10350 1900 0    50   ~ 0
+CAN_EN
+Text Label 10350 1800 0    50   ~ 0
+CAN_SILENT
+Wire Wire Line
+	9800 1600 10800 1600
+$Comp
+L Interface_CAN_LIN:MCP2515-xSO U?
+U 1 1 5F40DB1B
+P 9200 2100
+F 0 "U?" H 8900 2850 50  0000 C CNN
+F 1 "MCP2515-xSO" H 9500 2850 50  0000 C CNN
+F 2 "Package_SO:SOIC-18W_7.5x11.6mm_P1.27mm" H 9200 1200 50  0001 C CIN
+F 3 "http://ww1.microchip.com/downloads/en/DeviceDoc/21801e.pdf" H 9300 1300 50  0001 C CNN
+	1    9200 2100
+	1    0    0    -1
+$EndComp
+$Comp
+L power:VCC #PWR?
+U 1 1 5F161781
+P 10400 4350
+F 0 "#PWR?" H 10400 4200 50  0001 C CNN
+F 1 "VCC" H 10415 4523 50  0000 C CNN
+F 2 "" H 10400 4350 50  0001 C CNN
+F 3 "" H 10400 4350 50  0001 C CNN
+	1    10400 4350
+	1    0    0    -1
+$EndComp
+$Comp
+L power:VCC #PWR?
+U 1 1 5F16C50B
+P 11400 3800
+F 0 "#PWR?" H 11400 3650 50  0001 C CNN
+F 1 "VCC" H 11415 3973 50  0000 C CNN
+F 2 "" H 11400 3800 50  0001 C CNN
+F 3 "" H 11400 3800 50  0001 C CNN
+	1    11400 3800
+	1    0    0    -1
+$EndComp
+$Comp
+L power:VCC #PWR?
+U 1 1 5F16D779
+P 10750 2300
+F 0 "#PWR?" H 10750 2150 50  0001 C CNN
+F 1 "VCC" H 10765 2473 50  0000 C CNN
+F 2 "" H 10750 2300 50  0001 C CNN
+F 3 "" H 10750 2300 50  0001 C CNN
+	1    10750 2300
+	1    0    0    -1
+$EndComp
+$Comp
+L power:VCC #PWR?
+U 1 1 5F16D998
+P 8450 3100
+F 0 "#PWR?" H 8450 2950 50  0001 C CNN
+F 1 "VCC" H 8465 3273 50  0000 C CNN
+F 2 "" H 8450 3100 50  0001 C CNN
+F 3 "" H 8450 3100 50  0001 C CNN
+	1    8450 3100
+	1    0    0    -1
+$EndComp
+$Comp
+L power:VCC #PWR?
+U 1 1 5F178A75
+P 9200 1200
+F 0 "#PWR?" H 9200 1050 50  0001 C CNN
+F 1 "VCC" H 9215 1373 50  0000 C CNN
+F 2 "" H 9200 1200 50  0001 C CNN
+F 3 "" H 9200 1200 50  0001 C CNN
+	1    9200 1200
+	1    0    0    -1
+$EndComp
+$Comp
+L power:VCC #PWR?
+U 1 1 5F17982A
+P 11300 1200
+F 0 "#PWR?" H 11300 1050 50  0001 C CNN
+F 1 "VCC" H 11315 1373 50  0000 C CNN
+F 2 "" H 11300 1200 50  0001 C CNN
+F 3 "" H 11300 1200 50  0001 C CNN
+	1    11300 1200
+	1    0    0    -1
+$EndComp
+Wire Wire Line
+	11300 1200 11300 1300
+Wire Wire Line
+	9200 1200 9200 1300
+Wire Wire Line
+	10750 2300 10750 2400
+Wire Wire Line
+	8450 3100 8450 3200
+Wire Wire Line
+	11400 3800 11400 3900
+Wire Wire Line
+	10400 4350 10400 4450
+$Comp
+L power:GND #PWR?
+U 1 1 5F1D2FBA
+P 8450 3500
+F 0 "#PWR?" H 8450 3250 50  0001 C CNN
+F 1 "GND" H 8455 3327 50  0000 C CNN
+F 2 "" H 8450 3500 50  0001 C CNN
+F 3 "" H 8450 3500 50  0001 C CNN
+	1    8450 3500
+	1    0    0    -1
+$EndComp
+$Comp
+L power:GND #PWR?
+U 1 1 5F1D5C54
+P 10750 2700
+F 0 "#PWR?" H 10750 2450 50  0001 C CNN
+F 1 "GND" H 10755 2527 50  0000 C CNN
+F 2 "" H 10750 2700 50  0001 C CNN
+F 3 "" H 10750 2700 50  0001 C CNN
+	1    10750 2700
+	1    0    0    -1
+$EndComp
+$Comp
+L Device:C_Small C?
+U 1 1 5F0DAE10
+P 11400 4000
+F 0 "C?" H 11492 4046 50  0000 L CNN
+F 1 "0.1uF" H 11492 3955 50  0000 L CNN
+F 2 "" H 11400 4000 50  0001 C CNN
+F 3 "~" H 11400 4000 50  0001 C CNN
+	1    11400 4000
+	1    0    0    -1
+$EndComp
+$Comp
+L power:GND #PWR?
+U 1 1 5F1D6D16
+P 11400 4200
+F 0 "#PWR?" H 11400 3950 50  0001 C CNN
+F 1 "GND" H 11405 4027 50  0000 C CNN
+F 2 "" H 11400 4200 50  0001 C CNN
+F 3 "" H 11400 4200 50  0001 C CNN
+	1    11400 4200
+	1    0    0    -1
+$EndComp
+$Comp
+L power:GND #PWR?
+U 1 1 5F1E188C
+P 10400 5950
+F 0 "#PWR?" H 10400 5700 50  0001 C CNN
+F 1 "GND" H 10405 5777 50  0000 C CNN
+F 2 "" H 10400 5950 50  0001 C CNN
+F 3 "" H 10400 5950 50  0001 C CNN
+	1    10400 5950
+	1    0    0    -1
+$EndComp
+Wire Wire Line
+	10400 5850 10400 5950
+Wire Wire Line
+	11400 4100 11400 4200
+Wire Wire Line
+	10750 2600 10750 2700
+Wire Wire Line
+	8450 3400 8450 3500
+Wire Wire Line
+	11300 2100 11300 2200
+$Comp
+L power:GND #PWR?
+U 1 1 5F210B66
+P 11300 2200
+F 0 "#PWR?" H 11300 1950 50  0001 C CNN
+F 1 "GND" H 11305 2027 50  0000 C CNN
+F 2 "" H 11300 2200 50  0001 C CNN
+F 3 "" H 11300 2200 50  0001 C CNN
+	1    11300 2200
+	1    0    0    -1
+$EndComp
+$Comp
+L power:GND #PWR?
+U 1 1 5F26891B
+P 9200 3000
+F 0 "#PWR?" H 9200 2750 50  0001 C CNN
+F 1 "GND" H 9205 2827 50  0000 C CNN
+F 2 "" H 9200 3000 50  0001 C CNN
+F 3 "" H 9200 3000 50  0001 C CNN
+	1    9200 3000
+	1    0    0    -1
+$EndComp
+Wire Wire Line
+	9200 2900 9200 3000
 $EndSCHEMATC

Commit message: Sync commit
Parts:
- removed U?: ATtiny814-SS, Package_SO:SOIC-14_3.9x8.7mm_P1.27mm, symbol MCU_Microchip_ATtiny:ATtiny814-SS
- added C? (x2): 33pF, symbol Device:C_Small
- added J?: Conn_02x03_Top_Bottom, symbol Connector_Generic:Conn_02x03_Top_Bottom
- added R?: 68k, symbol Device:R_Small_US
- added R?: 4.7k, symbol Device:R_US
- added R? (x2): NP, symbol Device:R_Small
- added R? (x2): 68k, symbol Device:R_Small
- added U?: ATtiny3216-S, Package_SO:SOIC-20W_7.5x12.8mm_P1.27mm, symbol MCU_Microchip_ATtiny:ATtiny3216-S
- added Y?: 20MHz/20pF, symbol Device:Crystal
Connections:
- net BREAKn: now also U?.10 (PB1)
- net CAN_EN: now also U?.5 (EN), U?.13 (PC1); no longer U?.8 (S)
- net CAN_SILENT: now also U?.8 (S), U?.12 (PC0); no longer U?.5 (EN)
- net DIR: now also U?.11 (PB0)
- net ENABLE: now also U?.8 (PB3)
- net GND: now also C?.2, C?.2, J?.3 (Pin_3), R?.2, R?.2, R?.2, U?.20 (GND)
- net HALL_A: now also U?.5 (PA7)
- net HALL_B: now also U?.3 (PA5)
- net HALL_C: now also U?.2 (PA4)
- net SPI_MISO: now also U?.18 (PA2)
- net SPI_MOSI: now also U?.17 (PA1)
- net SPI_SCK: now also U?.19 (PA3)
- net VCC: now also J?.4 (Pin_4), R?.1, R?.1, U?.1 (VCC); no longer U7.19 (Speed)
- net MOTOR_FAULT: now reaches D1.2 (A), R13.2, U7.22 (Fault)
- net MOTOR_FAULT: now also U?.9 (PB2)
- net CAN_RXINT1n: now reaches U?.10 (~RX1BF)
- net CAN_RXINT0n: now reaches U?.11 (~RX0BF)
- net CAN_INTn: now reaches U?.12 (~INT)
- net CAN_INTn: now also U?.15 (PC3)
- net CAN_CSn: now reaches U?.16 (~CS)
- net CAN_CSn: now also U?.14 (PC2)
- net CAN_RSTn: now reaches U?.17 (~RESET)
- net CAN_RSTn: now also R?.1
- net CAN_CLK: now reaches U?.3 (CLKOUT/SOF)
- net CRY_OSC2: now reaches U?.7 (OSC2)
- net CRY_OSC2: now also C?.1, Y?.1
- net CRY_OSC1: now reaches U?.8 (OSC1)
- net CRY_OSC1: now also C?.1, Y?.2
- new net CAN_ID0: R?.1, R?.2, U?.7 (PB4)
- new net CAN_ID1: R?.1, R?.2, U?.6 (PB5)
- new net SPEED: U7.19 (Speed), U?.4 (PA6)
- new net UPDI_RX: J?.2 (Pin_2), R?.2, U?.16 (~RESET~/PA0)
- new net UPDI_TX: J?.1 (Pin_1), R?.1
- no-connect marks 0 -> 3
Other:
- note added: "Bridge Pads to change ID"
- note added: "CAN ID select"
- note added: "Microcontroller and Configuration"
- note added: "TODO I don't like high and low current voltages on same connector"
- note added: "TODO pick fault LED and resize resistor\n"
- note removed: "TODO resistor too small?"
- moved on the sheet: C?, J4, J?, R?
